File: zeitgeist.brd (EAGLE design)
At the start: 110 x 85 mm, 86 parts, among them IC1 78L05, SW1 SUBMINI_SPDT, SW2 SUBMINI_SPDT, T2 2N3904, U2 TL074P, U3 PT2399DIL16

Commit message: Fixed reversed Time and Mod pots
Parts:
- moved P1 28.5 mm to (40.0, 59.0)
- moved P2 28.5 mm to (11.5, 59.0)
- turned R23 to 0 degrees
Routing:
- net CV_OUT: track 55.3 -> 33.3 mm, vias 1 -> 0
- net N$35: track 6.26 -> 28.2 mm
- net N$32: track 3.42 -> 23.7 mm, vias 0 -> 1
- net N$34: track 62.3 -> 68.0 mm
- net N$39: track 55.2 -> 52.2 mm
- net N$12: track 108.6 -> 110.3 mm
- net DELAY_OUT: track 76.2 -> 77.6 mm
Other:
- board text added: "ROB HORDIJK ZEITGEIST V1.1 June 2023"
- board text removed: "ROB HORDIJK ZEITGEIST V1.0 May 2023"
